File: live_telemetry/telemetry_receiver/telemetry_receiver.kicad_pcb (KiCad board)
At the start: 2 copper layers, 45.7 x 28 mm, 21 parts, among them J1 Conn_Coaxial, J2 Programming Header, J3 USB_A, U1 PIC16LF1455, U2 RFM95W, U3 AP2114H-3.3

Commit message: Update schematics and silkscreens to fix issues from assembly
Other:
- board text added: "Kyoto Telemetry RX D. Kletke 2020-02-23"
- board text removed: "Kyoto D. Kletke 2020-02-23"
Changed lines of the file:
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@@
     )
   )
-  (gr_text "Kyoto\nD. Kletke\n2020-02-23" (at 137.4902 97.7646) (layer B.SilkS)
+  (gr_text "Kyoto\nTelemetry RX\nD. Kletke\n2020-02-23" (at 137.4902 97.7646) (layer B.SilkS)
     (effects (font (size 1 1) (thickness 0.15)) (justify mirror))
   )
